File: ESP/AutoProgramFTDI/AutoProgramFTDI.brd (EAGLE design)
At the start: 26.4 x 17.3 mm, 21 parts, among them U2 CH340G, U4 74LVC1G08SE, Y1 12MHz

Commit message: update usb & Arduino pro mini
Parts:
- removed X1: (no value), Scott-Connectors:MICROUSB_4UCONN_20329_V2
- added U$9: USB_ON_BOARD, Scott-Connectors:USB_ON_BOARD
Connections:
- net 5V: now also U$9.VCC; no longer X1.VBUS
- net GND: now also U$9.GND; no longer X1.BASE@1, X1.BASE@2, X1.GND, X1.SPRT@1, X1.SPRT@2, X1.SPRT@3, X1.SPRT@4
- net N$6: now also U$9.D-; no longer X1.D-
- net N$7: now also U$9.D+; no longer X1.D+
Routing:
- net GND: track 65.4 -> 0.00 mm, vias 3 -> 0
- net 3.3V: track 59.1 -> 0.00 mm, vias 3 -> 0
- net N$1: track 46.5 -> 0.00 mm, vias 2 -> 0
- net RXI: track 38.9 -> 0.00 mm, vias 2 -> 0
- net !DTR: track 38.8 -> 0.00 mm, vias 1 -> 0
- net !RTS: track 35.0 -> 0.00 mm, vias 5 -> 0
- net TXO: track 35.0 -> 0.00 mm, vias 1 -> 0
- net N$9: track 26.6 -> 0.00 mm, vias 4 -> 0
- net N$2: track 25.4 -> 0.00 mm, vias 2 -> 0
- net N$8: track 20.9 -> 0.00 mm
- net 5V: track 18.3 -> 0.00 mm, vias 1 -> 0
- net N$6: track 10.4 -> 0.00 mm
- net N$7: track 10.4 -> 0.00 mm
- net IO0: track 9.79 -> 0.00 mm
- net N$3: track 7.80 -> 0.00 mm
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