File: ESP/ESP12Breakout/ESP_Breakout.sch (EAGLE design)
At the start: 15 parts, among them U1 AMS1117-3.3, X2 ESP-12

Commit message: update usb & Arduino pro mini
Parts:
- removed BATT: BATTERY_THD_+-, AutoPark:BATTERY_THD_+-
- removed ESP_PRGM: JST_1.25_6P, Scott-Connectors:JST_1.25_6P
- removed FTDI: (no value), pinhead:PINHD-1X6
- removed PRGM: PUSHBUTTON, AutoPark:PUSHBUTTON
- added PROGRAMMER: JST_1.25_6P, Scott-Connectors:JST_1.25_6P
- R2: value 4.7K -> 330
Connections:
- new net N$2: LED.DI, R2.2
- net 3.3V: now also PROGRAMMER.6; no longer ESP_PRGM.1, FTDI.1, RN1.1
- net GND: now also PROGRAMMER.5, RN1.1; no longer BATT.-, ESP_PRGM.2, FTDI.2, PRGM.1, R2.1
- net GPIO0: now also PROGRAMMER.1; no longer ESP_PRGM.6, PRGM.2, RN1.7
- net GPIO15: now also R2.1, RN1.8; no longer LED.DI, R2.2
- net N$1: no longer BATT.+
- net RESET: now also PROGRAMMER.2, RN1.7; no longer ESP_PRGM.5, RN1.8
- net RXD: now also PROGRAMMER.4; no longer ESP_PRGM.4
- net TXD: now also PROGRAMMER.3; no longer ESP_PRGM.3, FTDI.4
- net USB_RX: no longer FTDI.3
Other:
- note removed: "There should be a 470R in series between DI and GPIO15!"
- moved on the sheet: R2, RESET
