File: Projects/MCU/STM32/STM32F303VC_linefollow/LineFollowTest.brd (EAGLE design)
At the start: 55 x 47.8 mm, 36 parts, among them J4 USB-MICRO-B-SOCKET-2, X1 NX3225GD-8MHZ

Commit message: bump 2/22
Parts:
- added GND: THD_01, Scott-Connectors:1X01
- added PHOTO: (no value), SparkFun-Connectors:1X04
- added R10: 1.5K, Scott-Electrical:0603
- added R12: 10k, Scott-Electrical:RESCAF80P320X160X60-8N
- added R13: 100, Scott-Electrical:RESCAF80P320X160X60-8N
- added U5, U6, U7, U8: QRE1113, Scott-Sensors:QRE1113-W
- C13, C14: value 10p -> 20p
- R7: value 390 -> 220
- renumbered U$1 to STM32F303
Connections:
- new net N$13: R13.1, U5.1
- new net N$14: R13.2, U6.1
- new net N$15: R13.3, U7.1
- new net N$16: R13.4, U8.1
- new net OUT1: PHOTO.1, R12.4, U5.3
- new net OUT2: PHOTO.2, R12.3, U6.3
- new net OUT3: PHOTO.3, R12.2, U7.3
- new net OUT4: PHOTO.4, R12.1, U8.3
- net 3V3: now also R10.1, R12.5, R12.6, R12.7, R12.8, R13.5, R13.6, R13.7, R13.8
- net GND: now also GND.1, U5.2, U5.4, U6.2, U6.4, U7.2, U7.4, U8.2, U8.4
- net N$12: now also R10.2
Routing:
- net 3V3: track 114.1 -> 166.4 mm, vias 7 -> 9
- net OUT4: track 0.00 -> 18.6 mm
- net OUT1: track 0.00 -> 14.8 mm
- net N$13: track 0.00 -> 13.7 mm
- net OUT3: track 0.00 -> 11.4 mm
- net N$16: track 0.00 -> 9.88 mm
- net OUT2: track 0.00 -> 9.03 mm
- net N$14: track 0.00 -> 7.06 mm
- net N$15: track 0.00 -> 4.70 mm
- net N$12: track 4.05 -> 6.09 mm
Other:
- board size 55 x 47.8 mm -> 72.5 x 48.3 mm
- board text added: "STM32F3 ADC Test V2 Aug 30, 2019"
- board text removed: "STM32F3 ADC Test V1 Aug 20, 2019"
