File: Projects/MCU/STM32/STM32F303VC_linefollow/LineFollowTest.sch (EAGLE design)
At the start: 36 parts, among them J4 USB-MICRO-B-SOCKET-2, X1 NX3225GD-8MHZ

Commit message: bump 2/22
Parts:
- added GND: THD_01, Scott-Connectors:THD_01
- added PHOTO: (no value), SparkFun-Connectors:CONN_04PTH
- added R10: 1.5K, Scott-Electrical:RESISTOR0603
- added R12: 10k, Scott-Electrical:RESISTOR_ARRAY_1206_SEPARATE
- added R13: 100, Scott-Electrical:RESISTOR_ARRAY_1206_SEPARATE
- added U5, U6, U7, U8: QRE1113, Scott-Sensors:QRE1113SMD-W
- C13, C14: value 10p -> 20p
- R7: value 390 -> 220
- renumbered U$1 to STM32F303
Connections:
- new net N$13: R13@1.1, U5.A
- new net N$14: R13@2.1, U6.A
- new net N$15: R13@3.1, U7.A
- new net N$16: R13@4.1, U8.A
- new net OUT1: PHOTO.1, R12@4.1, U5.C
- new net OUT2: PHOTO.2, R12@3.1, U6.C
- new net OUT3: PHOTO.3, R12@2.1, U7.C
- new net OUT4: PHOTO.4, R12@1.1, U8.C
- net 3V3: now also R10.1, R12@1.2, R12@2.2, R12@3.2, R12@4.2, R13@1.2, R13@2.2, R13@3.2, R13@4.2
- net GND: now also GND.1, U5.E, U5.K, U6.E, U6.K, U7.E, U7.K, U8.E, U8.K
- net N$12: now also R10.2
Other:
- note added: "Aug 30, 2019 V2: Fix missing pull up USB V+"
- note added: "Revision History"
