File: Projects/MCU/ESP/ESP32Breakout/ESP32Breakout.brd (EAGLE design)
At the start: 22 parts, among them Q1 DMG3415U, SW2 KMR2, X2 ESP32_WROOM32

Commit message: esp32 dbl
Parts:
- removed SW2: KMR2, Scott-Switches:BTN_KMR2_4.6X2.8
- added J1: (no value), Scott-Electrical:0603
- added RST: KMR2, Scott-Switches:BTN_KMR2_4.6X2.8
- C1: value 10uF -> 0.1uF; device Scott-Electrical:CAP_0805 -> Scott-Electrical:0603
- C2: device Scott-Electrical:CAP_0805 -> Scott-Electrical:0805
- C3, C5: device Scott-Electrical:CAP_0603 -> Scott-Electrical:0603
- C4: device Scott-Electrical:CAP_0603 -> Scott-Electrical:0805
- C6: device Scott-Electrical:CAP_0805 -> Scott-Electrical:0603
- CHG: value ORANGE -> (none); device Scott-Electrical:MICROBUILDER_CHIPLED_0603 -> Scott-Electrical:CHIPLED_0603
- R1: value 4.7K -> 4.7k
- R2: value 1K -> 1k
- R3: value 10K -> 10k
- R4: value 330 -> (none)
- RA1: value 100K -> (none)
- moved R1 63.1 mm to (-26.7, 51.4), turned to 180 degrees
- moved X2 62.9 mm to (3.81, 62.7), turned to 0 degrees
- moved C1 62.5 mm to (-7.24, 66.9), turned to 90 degrees
- moved CHG 60.2 mm to (-26.7, 55.2), turned to 90 degrees
- moved MCP 59.4 mm to (-23.5, 52.2), turned to 0 degrees
- moved BAT 59.2 mm to (-27.2, 63.1), turned to 90 degrees
- moved R2 57.1 mm to (-26.7, 53.5)
- moved Q1 56.1 mm to (-19.8, 50.9), turned to 90 degrees
- moved D1 56.0 mm to (-17.0, 51.1), turned to 270 degrees
- moved C5 55.5 mm to (-10.0, 57.3), turned to 0 degrees
- moved C6 54.0 mm to (-10.0, 59.3), turned to 0 degrees
- moved RA1 53.0 mm to (-9.91, 49.9), turned to 0 degrees
- moved C2 52.6 mm to (-19.8, 55.1), turned to 0 degrees
- moved REG 49.3 mm to (-9.91, 54.2), turned to 0 degrees
- moved C4 48.2 mm to (-12.8, 52.1), turned to 270 degrees
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Connections:
- net A13_I35: now also RA1.4, RA1.6; no longer RA1.3, RA1.8
- net EN: now also RA1.8; no longer RA1.2
- net GND: now also RA1.5, RA1.7, RST.A, RST.A'; no longer RA1.1, RA1.4, SW2.A, SW2.A'
- net N$7: now also J1.2, RA1.1; no longer RA1.6
- net RESET: now also RST.B, RST.B'; no longer SW2.B, SW2.B'
- net VBAT: now also RA1.3; no longer RA1.7
- net VBUS: now also J1.1, RA1.2; no longer RA1.5
Routing:
- net 3.3V: track 0.00 -> 60.6 mm, vias 0 -> 2
- net RESET: track 0.00 -> 46.6 mm, vias 0 -> 2
- net VBUS: track 0.00 -> 46.4 mm
- net VBAT: track 0.00 -> 31.1 mm, vias 0 -> 2
- net TXD0: track 0.00 -> 22.9 mm, vias 0 -> 2
- net RXD0: track 0.00 -> 22.8 mm, vias 0 -> 2
- net A13_I35: track 0.00 -> 15.7 mm
- net N$7: track 0.00 -> 10.4 mm
- net IO13_A12: track 0.00 -> 8.24 mm
- net GPIO0: track 0.00 -> 7.02 mm
- net N$3: track 0.00 -> 6.84 mm
- net N$2: track 0.00 -> 4.08 mm
- net N$4: track 0.00 -> 2.63 mm
- net EN: track 0.00 -> 1.85 mm
- net N$1: track 0.00 -> 1.82 mm
Other:
- board text added: "3V3 Reg/Filter"
- board text added: "LiPo Charging"
- board text removed: "BOARD NAME"
- board text removed: "CHG"
- board text removed: "DATE"
- board text removed: "RST"
